File: design_files/AST1008.sch (EAGLE design)
At the start: 7 parts, among them J1 SM05B, U1 TSOP57438

Commit message: updated documentation
Parts:
- C2: value 10uF -> 1uF; device tinycircuits:AS-ITM-00002 -> tinycircuits:AS-ITM-00410; PARTNO (none) -> AS-ITM-00410; VALUE (none) -> 1uF
- J1: device tinycircuits:AS-ITM-00340 -> tinycircuits:AS-ITM-00340EDGE
- R1, R3: value 0.0 -> 1.00K; device tinycircuits:AS-ITM-00076 -> tinycircuits:AS-ITM-00003; PARTNO AS-ITM-00076 -> AS-ITM-00003; VALUE 0.0 -> 1.00K
- R2: value 0.0 -> 1.00K; device tinycircuits:AS-ITM-00076 -> tinycircuits:AS-ITM-00003; PARTNO (none) -> AS-ITM-00003; VALUE (none) -> 1.00K
Connections:
- net INT: now also R1.2; no longer R2.2
- net SCL: now also R2.2; no longer R1.2
Other:
- note added: "38KHz Infrared Receiver"
- note added: "Hand Populated: -"
- note added: "Hand Soldered: -"
- note added: "Non Populated: R2, R3"
- note added: "Notes: -"
- note added: "Variant: Standard - R"
- note added: "Wireling IR Receiver"
- note removed: "Choose Receiver and Emitter Components"
- note removed: "InfraRed Board"
- note removed: "InfraRed Receiver Board"
- note removed: "NOTES:"
- note removed: "Optional Resistor Population for Data Signal"
- moved on the sheet: R1, R2
